File: hardware/pc_kalam32_dev_v1/pc_kalam32_dev.brd (EAGLE design)
At the start: 68.6 x 53.3 mm, 86 parts, among them Q3 2.5A/30V, Q5 MBT3904DW1T1, U1 AP2112K-3.3V, U10 ESP3212, U4 FTS31XS-U, U5 MCP73831, U6 W25Q32FVSS, Y2 26MHz, Y3 32.768kHz

Commit message: Updated schematics
Parts:
- removed U$3: KALAM32-DEV, circuitects:KALAM32-DEV
- removed U$4: PROTY_LOGO_WITH_TEXT, circuitects:PROTY_WITH_TEXT
Connections:
- net 15 renamed TOUCH/15
- net 4 renamed TOUCH/4
- removed net AIN0: AD.4, U10.20
- removed net AIN1: AD.3, U10.18
- removed net WS2812_LED: R1.2, U10.11
- new net AIN0/34: AD.4, U10.10
- new net AIN1/35: AD.3, U10.11
- new net WS2812/13: R1.2, U10.20
- net 36: no longer IOL.1
- net 37: no longer IOL.2
- net 38: no longer IOL.4
- net 39: no longer IOL.3
- net SS: now also U10.18; no longer U10.10
Routing:
- net 36: track 99.0 -> 11.9 mm, vias 3 -> 2
- net 37: track 96.3 -> 9.94 mm, vias 3 -> 2
- net 38: track 91.3 -> 18.4 mm, vias 3 -> 2
- net AIN0: track 55.8 -> 0.00 mm, vias 1 -> 0
- net AIN0/34: track 0.00 -> 54.8 mm, vias 0 -> 1
- net AIN1: track 51.6 -> 0.00 mm, vias 1 -> 0
- net AIN1/35: track 0.00 -> 50.3 mm, vias 0 -> 1
- net WS2812_LED: track 48.8 -> 0.00 mm, vias 2 -> 0
- net 39: track 92.8 -> 48.4 mm, vias 3 -> 2
- net VUSB: track 132.0 -> 130.7 mm
- net TOUCH/15: track 21.5 -> 20.7 mm
- net SS: track 57.9 -> 57.2 mm
- net TOUCH/4: track 49.9 -> 49.3 mm

Commit message: added design file for v1.1
Parts:
- moved U$12 78.1 mm to (52.4, 35.7), flipped to the bottom
- moved U$13 31.1 mm to (25.6, 0.90), flipped to the bottom
- moved R29 0.32 mm to (23.6, 22.5)
- moved Y3 0.22 mm to (20.5, 20.9)
- moved C43 0.20 mm to (21.4, 23.7)
- moved C41 0.10 mm to (21.7, 25.0)
- moved C42 0.10 mm to (21.3, 18.4)
Connections:
- net 25 renamed DAC1/GPIO25
- net 26 renamed DAC2/GPIO26
- net MISO renamed MISO/GPIO19
- net MOSI renamed MOSI/GPIO23
- net SCK renamed SCK/GPIO18
- net SCL renamed SCL/GPIO22
- net SDA renamed SDA/GPIO21
- net SS renamed CS/GPIO12
- removed net 36: C19.2, U10.5
- removed net 39: C20.2, U10.8
- removed net AIN0/34: AD.4, U10.10
- removed net AIN1/35: AD.3, U10.11
- removed net AIN2: AD.2, U10.17
- removed net AIN3: AD.1, U10.16
- removed net WS2812/13: R1.2, U10.20
- new net ADC1:0/GPI36: AD.3, C19.2, U10.5
- new net ADC1:3/GPI39: AD.4, C20.2, U10.8
- new net ADC1:6/GPI34: AD.2, U10.10
- new net ADC1:7/GPI35: AD.1, U10.11
- new net GP14: IOL.2, U10.17
- new net GP27: IOL.1, U10.16
- new net WS2812/GPIO13: IOL.3, R1.2, U10.20
- net 17: now also IOL.8; no longer IOH.2
- net VBAT: now also POWER.5
Routing:
- net GP27: track 0.00 -> 89.3 mm, vias 0 -> 1
- net GP14: track 0.00 -> 87.8 mm, vias 0 -> 1
- net WS2812/GPIO13: track 0.00 -> 63.5 mm, vias 0 -> 3
- net ADC1:0/GPI36: track 0.00 -> 56.5 mm, vias 0 -> 2
- net ADC1:3/GPI39: track 0.00 -> 55.8 mm, vias 0 -> 2
- net AIN0/34: track 54.8 -> 0.00 mm, vias 1 -> 0
- net ADC1:6/GPI34: track 0.00 -> 52.1 mm, vias 0 -> 2
- net AIN1/35: track 50.3 -> 0.00 mm, vias 1 -> 0
- net ADC1:7/GPI35: track 0.00 -> 48.6 mm, vias 0 -> 2
- net 39: track 48.4 -> 0.00 mm, vias 2 -> 0
- net AIN2: track 48.3 -> 0.00 mm, vias 1 -> 0
- net AIN3: track 45.4 -> 0.00 mm, vias 1 -> 0
- net VBAT: track 12.4 -> 34.1 mm
- net 36: track 11.9 -> 0.00 mm, vias 2 -> 0
- net CS/GPIO12: track 57.2 -> 47.2 mm
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Other:
- board text added: "ADC1:0/GPI36"
- board text added: "ADC1:3/GPI39"
- board text added: "ADC1:6/GPI34"
- board text added: "ADC1:7/GPI35"
- board text added: "All Analog and Digital I/Os 3.3v ONLY"
- board text added: "CS/GPIO12"
- board text added: "DAC1/GPIO25"
- board text added: "DAC2/GPIO26"
- board text added: "GPIO14"
- board text added: "GPIO16"
- board text added: "GPIO17"
- board text added: "GPIO2"
- board text added: "GPIO27"
- board text added: "GPIO5"
- board text added: "Get Started: http://protocentral.com/kalam32"
- board text added: "LED_RX"
- board text added: "LED_TX"
- board text added: "MADE IN INDIA"
- board text added: "MISO/GPIO19"
- board text added: "MOSI/GPIO23"
- board text added: "NC"
- board text added: "PWR"
- board text added: "SCK/GPIO18"
- board text added: "SCL/GPIO22"
- board text added: "SDA/GPIO21"
- board text added: "SPI ONLY"
- board text added: "SW1/ GPIO0"
- board text added: "T1"
- board text added: "T2"
- board text added: "VBAT"
- board text added: "WS2812/GPIO13"
- board text added: "v1.1"
- board text removed: "3"
- board text removed: "9"
- board text removed: "POWER"
- board text removed: "SW1"
- board text removed: "To get started: http://protocentral.com/kalam32"
- board text removed: "v1"
