File: hardware/pc_kalam32_dev_v1/pc_kalam32_dev.sch (EAGLE design)
At the start: 84 parts, among them Q3 2.5A/30V, Q5 MBT3904DW1T1, U1 AP2112K-3.3V, U10 ESP3212, U4 FTS31XS-U, U5 MCP73831, U6 W25Q32FVSS, Y2 26MHz, Y3 32.768kHz

Commit message: Updated schematics
Parts:
- removed U$3: KALAM32-DEV, circuitects:KALAM32-DEV
- removed U$4: PROTY_LOGO_WITH_TEXT, circuitects:PROTY_LOGO_WITH_TEXT
Connections:
- net 15 renamed TOUCH/15
- net 4 renamed TOUCH/4
- removed net AIN0: AD.4, U10.(GPIO13/ADC2:4/TOUCH4/RTC14/SPID/U0CTS)MTCK
- removed net AIN1: AD.3, U10.(GPIO12/ADC2:5/TOUCH5/RTC15/SPIQ)MTDI
- removed net WS2812_LED: R1.2, U10.VDET_2(GPI35/ADC1:7)
- new net AIN0/34: AD.4, U10.VDET_1(GPI34/ADC1:6)
- new net AIN1/35: AD.3, U10.VDET_2(GPI35/ADC1:7)
- new net WS2812/13: R1.2, U10.(GPIO13/ADC2:4/TOUCH4/RTC14/SPID/U0CTS)MTCK
- net 36: no longer IOL.1
- net 37: no longer IOL.2
- net 38: no longer IOL.4
- net 39: no longer IOL.3
- net SS: now also U10.(GPIO12/ADC2:5/TOUCH5/RTC15/SPIQ)MTDI; no longer U10.VDET_1(GPI34/ADC1:6)
Other:
- note added: "Power"
- note added: "WS2812B LEDs"
- note removed: "JST"
- note removed: "SJ1 can be cut to disable the power LED. (Saving lots of power.)"

Commit message: added design file for v1.1
Connections:
- net 25 renamed DAC1/GPIO25
- net 26 renamed DAC2/GPIO26
- net MISO renamed MISO/GPIO19
- net MOSI renamed MOSI/GPIO23
- net SCK renamed SCK/GPIO18
- net SCL renamed SCL/GPIO22
- net SDA renamed SDA/GPIO21
- net SS renamed CS/GPIO12
- removed net 36: C19.2, U10.SENSOR_VP(GPI36/ADC1:0/RTC0)
- removed net 39: C20.2, U10.SENSOR_VN(GPI39/ADC1:3/RTC3)
- removed net AIN0/34: AD.4, U10.VDET_1(GPI34/ADC1:6)
- removed net AIN1/35: AD.3, U10.VDET_2(GPI35/ADC1:7)
- removed net AIN2: AD.2, U10.(GPIO14/ADC2:6/TOUCH6/RTC16/SPICLK)MTMS
- removed net AIN3: AD.1, U10.(ADC2:7/TOUCH7/RTC17)GPIO27
- removed net WS2812/13: R1.2, U10.(GPIO13/ADC2:4/TOUCH4/RTC14/SPID/U0CTS)MTCK
- new net ADC1:0/GPI36: AD.3, C19.2, U10.SENSOR_VP(GPI36/ADC1:0/RTC0)
- new net ADC1:3/GPI39: AD.4, C20.2, U10.SENSOR_VN(GPI39/ADC1:3/RTC3)
- new net ADC1:6/GPI34: AD.2, U10.VDET_1(GPI34/ADC1:6)
- new net ADC1:7/GPI35: AD.1, U10.VDET_2(GPI35/ADC1:7)
- new net GP14: IOL.2, U10.(GPIO14/ADC2:6/TOUCH6/RTC16/SPICLK)MTMS
- new net GP27: IOL.1, U10.(ADC2:7/TOUCH7/RTC17)GPIO27
- new net WS2812/GPIO13: IOL.3, R1.2, U10.(GPIO13/ADC2:4/TOUCH4/RTC14/SPID/U0CTS)MTCK
- net 17: now also IOL.8; no longer IOH.2
- net VBAT: now also POWER.5
